File: PCB_Kicad/Autoscope/Autoscope.kicad_pcb (KiCad board)
At the start: 2 copper layers, 85 x 56 mm, 42 parts, among them J1 Conn_01x02, J10 Conn_02x02_Odd_Even, J11 Conn_02x02_Odd_Even, J12 Conn_02x02_Odd_Even, J13 Conn_01x02, J2 Conn_01x02, J3 Conn_01x02, J4 Conn_01x02, J5 Conn_01x02, J6 12VDC Supply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

Commit message: refactor labels & fix a bug : invert GPS_EN GPS_Rx
Connections:
- net /Motor1_1A renamed /MotorE_1A
- net /Motor1_1B renamed /MotorE_1B
- net /Motor1_2A renamed /MotorE_2A
- net /Motor1_2B renamed /MotorE_2B
- net /Motor1_DIR renamed /MotorE_DIR
- net /Motor1_EN renamed /MotorE_EN
- net /Motor1_MS1 renamed /MotorE_MS1
- net /Motor1_MS2 renamed /MotorE_MS2
- net /Motor1_MS3 renamed /MotorE_MS3
- net /Motor1_STEP renamed /MotorE_STEP
- net /Motor2_1A renamed /MotorZ_1A
- net /Motor2_1B renamed /MotorZ_1B
- net /Motor2_2A renamed /MotorZ_2A
- net /Motor2_2B renamed /MotorZ_2B
- net /Motor2_DIR renamed /MotorZ_DIR
- net /Motor2_EN renamed /MotorZ_EN
- net /Motor2_MS1 renamed /MotorZ_MS1
- net /Motor2_MS2 renamed /MotorZ_MS2
- net /Motor2_MS3 renamed /MotorZ_MS3
- net /Motor2_STEP renamed /MotorZ_STEP
- net /Motor3_1A renamed /MotorA_1A
- net /Motor3_1B renamed /MotorA_1B
- net /Motor3_2A renamed /MotorA_2A
- net /Motor3_2B renamed /MotorA_2B
- net /Motor3_DIR renamed /MotorA_DIR
- net /Motor3_EN renamed /MotorA_EN
- net /Motor3_MS1 renamed /MotorA_MS1
- net /Motor3_MS2 renamed /MotorA_MS2
- net /Motor3_MS3 renamed /MotorA_MS3
- net /Motor3_STEP renamed /MotorA_STEP
- net /Position_sensor_1 renamed /Position_sensor_A1
- net /Position_sensor_2 renamed /Position_sensor_E2
- net /Position_sensor_3 renamed /Position_sensor_E1
- net /Position_sensor_4 renamed /Position_sensor_Z2
- net /Position_sensor_5 renamed /Position_sensor_Z1
- J8 pad 10: /GPS_EN -> /GPS_Rx
- J8 pad 7: /GPS_Rx -> /GPS_EN
- J9 pad 1: /GPS_EN -> /GPS_Rx
- J9 pad 3: /GPS_Rx -> /GPS_EN
Routing:
- net /GPS_Rx: track 30.2 -> 39.7 mm
- net /GPS_EN: track 39.7 -> 30.2 mm
